File: pcb/esp32s3_watches/power.kicad_sch (KiCad schematic)
At the start: 16 parts, among them J1 Barrel_Jack_MountingPin, J3 Screw_Terminal_01x02, U5 TLV62569DBV

Commit message: BOM file updates. Scheme complete.
Parts:
- C300: renamed from C1; value 1u -> 1uF; footprint Capacitor_SMD:C_0603_1608Metric -> Capacitor_SMD:C_0805_2012Metric; Manufacturer Product Number CL10B105KP8NNNC -> CL21B105KBFNNNE
- C301: renamed from C2; value 1u -> 1uF; footprint Capacitor_SMD:C_0603_1608Metric -> Capacitor_SMD:C_0805_2012Metric; Manufacturer Product Number CL10B105KP8NNNC -> CL21B105KBFNNNE
- C302: renamed from C3; value 22u -> 22uF; Manufacturer Product Number CL21A226MQQNNNE -> CL21A226MAYNNNE
- C303: renamed from C4; value 22u -> 22uF; Manufacturer Product Number CL21A226MQQNNNE -> CL21A226MAYNNNE
- C304: renamed from C5; footprint Capacitor_SMD:C_0402_1005Metric -> Capacitor_SMD:C_0603_1608Metric
- D300: renamed from D1; Manufacturer Product Number (none) -> SBR3M30P1-7
- D301: renamed from D2; Manufacturer Product Number (none) -> SBR3M30P1-7
- D302: renamed from D3; footprint LED_SMD:LED_0603_1608Metric -> LED_THT:LED_D5.0mm; Manufacturer Hubei KENTO Elec -> (none); Manufacturer Product Number KT-0603R -> (none)
- J300: renamed from J1; Manufacturer Product Number (none) -> DC-005-A200
- J301: renamed from J3; Manufacturer Product Number (none) -> WJ500V-5.08-2P
- L300: renamed from L1; footprint Inductor_SMD:L_0402_1005Metric -> Inductor_SMD:L_0603_1608Metric; Manufacturer Product Number LQG15HS10NJ02D -> LQG18HN10NJ00D
- L301: renamed from L2; value 15u -> 15uH; footprint BlackPill:MWSA0603S -> esp32s3_watches:MWSA0603S
- R300: renamed from R2; value 100k -> 100kR; footprint Resistor_SMD:R_0402_1005Metric -> Resistor_SMD:R_0805_2012Metric; Manufacturer Product Number 0402WGF1003TCE -> 0805W8F1003T5E
- R301: renamed from R3; value 22k -> 22kR; footprint Resistor_SMD:R_0402_1005Metric -> Resistor_SMD:R_0805_2012Metric; Manufacturer Product Number 0402WGF2202TCE -> 0805W8F2202T5E
- R302: renamed from R4; value 1k -> 500R; footprint Resistor_SMD:R_0402_1005Metric -> Resistor_SMD:R_0805_2012Metric; Manufacturer UNI-ROYAL(Uniroyal Elec) -> Viking Tech; Manufacturer Product Number 0402WGF1001TCE -> ARG05FTC5000
- renumbered U5 to U300
Other:
- moved on the sheet: C300, C301, C302, C303, C304, D301, D302, J301, L300, L301, R300, R301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
