File: pcb/esp32s3_watches/esp32s3_watches.kicad_pcb (KiCad board)
At the start: 2 copper layers, 89 parts, among them J1 Barrel_Jack_MountingPin, J2 10067847-001RLF, J3 Screw_Terminal_01x02, U1 ESP32-S3-DevKitC, U4 SW_DPDT_XLX, U5 TLV62569DBV

Commit message: BOM file updates. Scheme complete.
Parts:
- added BT400: BC2032-E2, esp32s3_watches:MPD_BC2032-E2, F.Cu at (246.0, 83.9)
- added C100: 10uF, Capacitor_SMD:C_0805_2012Metric, F.Cu at (211.7, 47.5)
- added C101: 100nF, Capacitor_SMD:C_0603_1608Metric, F.Cu at (218.8, 40.3)
- added C103: 100nF, Capacitor_SMD:C_0603_1608Metric, F.Cu at (218.8, 42.8)
- added C400: 10uF, Capacitor_SMD:C_0805_2012Metric, F.Cu at (223.7, 59.2)
- added C401: 100nF, Capacitor_SMD:C_0603_1608Metric, F.Cu at (228.0, 59.0)
- added C402: 15pF, Capacitor_SMD:C_0603_1608Metric, F.Cu at (244.4, 96.4)
- added D100: PESD3V3L1BA,115, Diode_SMD:D_SOD-323, F.Cu at (232.5, 115.3)
- added D101: PESD3V3L1BA,115, Diode_SMD:D_SOD-323, F.Cu at (232.5, 103.5)
- added D102: PESD3V3L1BA,115, Diode_SMD:D_SOD-323, F.Cu at (232.5, 106.4)
- added D103: PESD3V3L1BA,115, Diode_SMD:D_SOD-323, F.Cu at (232.5, 109.4)
- added D104: PESD3V3L1BA,115, Diode_SMD:D_SOD-323, F.Cu at (232.5, 112.3)
- added D401: 1N4148, Diode_SMD:D_SOD-123, F.Cu at (224.4, 52.7)
- added D402: 1N4148, Diode_SMD:D_SOD-123, F.Cu at (224.4, 56.1)
- added J101: Conn_01x04_Pin, Connector_PinHeader_1.27mm:PinHeader_1x04_P1.27mm_Vertical, F.Cu at (236.7, 103.7)
- added J102: Conn_01x04_Pin, Connector_PinHeader_1.27mm:PinHeader_1x04_P1.27mm_Vertical, F.Cu at (240.8, 103.7)
- added J103: Conn_01x04_Pin, Connector_PinHeader_1.27mm:PinHeader_1x04_P1.27mm_Vertical, F.Cu at (245.0, 103.7)
- added L301: 15uH, esp32s3_watches:MWSA0603S, F.Cu at (214.5, 55.1)
- added R100: 10kR, Resistor_SMD:R_0805_2012Metric, F.Cu at (210.7, 43.4)
- added R101: 10kR, Resistor_SMD:R_0805_2012Metric, F.Cu at (210.7, 45.2)
- added R102: 10kR, Resistor_SMD:R_0805_2012Metric, F.Cu at (213.1, 39.9)
- added R103: 10kR, Resistor_SMD:R_0805_2012Metric, F.Cu at (213.1, 41.7)
- added R104: 500R, Resistor_SMD:R_0805_2012Metric, F.Cu at (213.1, 43.4)
- added R106: 10kR, Resistor_SMD:R_0805_2012Metric, F.Cu at (213.1, 45.2)
- added R107: 10kR, Resistor_SMD:R_0805_2012Metric, F.Cu at (215.6, 39.9)
- added R108: 10kR, Resistor_SMD:R_0805_2012Metric, F.Cu at (215.6, 41.7)
- added R109: 10kR, Resistor_SMD:R_0805_2012Metric, F.Cu at (215.6, 43.4)
- added R110: 10kR, Resistor_SMD:R_0805_2012Metric, F.Cu at (215.6, 45.2)
- added R15: 500R, Resistor_SMD:R_0805_2012Metric, F.Cu at (210.7, 39.9)
- added R16: 500R, Resistor_SMD:R_0805_2012Metric, F.Cu at (210.7, 41.7)
- added R400: 5k1R, Resistor_SMD:R_0805_2012Metric, F.Cu at (228.5, 51.9)
- added R401: 5k1R, Resistor_SMD:R_0805_2012Metric, F.Cu at (228.5, 53.7)
- added U400: PCF8563TS, Package_SO:MSOP-8_3x3mm_P0.65mm, F.Cu at (234.0, 97.7)
- added Y400: 32768Hz, Crystal:Crystal_SMD_3225-4Pin_3.2x2.5mm, F.Cu at (240.4, 97.6)
- C300: renamed from C1; value 1u -> 1uF; footprint Capacitor_SMD:C_0603_1608Metric -> Capacitor_SMD:C_0805_2012Metric
- C301: renamed from C2; value 1u -> 1uF; footprint Capacitor_SMD:C_0603_1608Metric -> Capacitor_SMD:C_0805_2012Metric
- C302: renamed from C3; value 22u -> 22uF
- C303: renamed from C4; value 22u -> 22uF
- C304: renamed from C5; footprint Capacitor_SMD:C_0402_1005Metric -> Capacitor_SMD:C_0603_1608Metric
- D302: renamed from D3; footprint LED_SMD:LED_0603_1608Metric -> LED_THT:LED_D5.0mm
- L300: renamed from L1; footprint Inductor_SMD:L_0402_1005Metric -> Inductor_SMD:L_0603_1608Metric
- R300: renamed from R2; value 100k -> 100kR; footprint Resistor_SMD:R_0402_1005Metric -> Resistor_SMD:R_0805_2012Metric
- R301: renamed from R3; value 22k -> 22kR; footprint Resistor_SMD:R_0402_1005Metric -> Resistor_SMD:R_0805_2012Metric
- R302: renamed from R4; value 1k -> 500R; footprint Resistor_SMD:R_0402_1005Metric -> Resistor_SMD:R_0805_2012Metric
- renumbered D64 to D105, D62 to D106, D63 to D107, D1 to D300, D2 to D301, J2 to J100, J1 to J300, J3 to J301, R1 to R105, U4 to SW100, SW1 to SW101, SW2 to SW102, SW3 to SW103, SW4 to SW104, U1 to U100, U3 to U101, Brd1 to U102, U2 to U103, U5 to U300
Connections:
- D105 pad 1: unconnected-(D64-K-Pad1) -> Net-(D105-K)
- D105 pad 2: unconnected-(D64-A-Pad2) -> Net-(D105-A)
- D106 pad 1: unconnected-(D62-K-Pad1) -> Net-(D106-K)
- D106 pad 2: unconnected-(D62-A-Pad2) -> LED_1
- D107 pad 1: unconnected-(D63-K-Pad1) -> Net-(D107-K)
- D107 pad 2: unconnected-(D63-A-Pad2) -> LED_2
- J100 pad 1: unconnected-(J2-DAT3/CD-Pad1) -> SD_CARD_CS
- J100 pad 2: unconnected-(J2-CMD-Pad2) -> SD_CARD_MOSI
- J100 pad 3: unconnected-(J2-VSS-Pad3) -> GND
- J100 pad 4: unconnected-(J2-VDD-Pad4) -> +3.3V
- J100 pad 5: unconnected-(J2-CLK-Pad5) -> SD_CARD_SCK
- J100 pad 6: unconnected-(J2-VSS__1-Pad6) -> GND
- J100 pad 7: unconnected-(J2-DAT0-Pad7) -> SD_CARD_MISO
- J100 pad G1: unconnected-(J2-GND-PadG1) -> GND
- J100 pad G2: unconnected-(J2-GND__1-PadG2) -> GND
- R105 pad 1: unconnected-(R1-Pad1) -> LDR_IN
- R105 pad 2: unconnected-(R1-Pad2) -> +3.3V
- SW100 pad 1: unconnected-(U4-Pad1) -> GND
- SW100 pad 2: unconnected-(U4-Pad2) -> /esp32-s3/LD2410_VCC
- SW100 pad 3: unconnected-(U4-Pad3) -> +5V
- SW100 pad 4: unconnected-(U4-Pad4) -> +5V
- SW100 pad 5: unconnected-(U4-Pad5) -> /esp32-s3/LD2410_VCC
- SW100 pad 6: unconnected-(U4-Pad6) -> GND
- SW101 pad 1: unconnected-(SW1-Pad1) -> +3.3V
- SW101 pad 2: unconnected-(SW1-Pad2) -> BUTTON_SW_1
- SW102 pad 1: unconnected-(SW2-Pad1) -> +3.3V
- SW102 pad 2: unconnected-(SW2-Pad2) -> BUTTON_SW_2
- SW103 pad 1: unconnected-(SW3-Pad1) -> +3.3V
- SW103 pad 2: unconnected-(SW3-Pad2) -> BUTTON_SW_3
- SW104 pad 1: unconnected-(SW4-Pad1) -> +3.3V
- SW104 pad 2: unconnected-(SW4-Pad2) -> BUTTON_SW_4
- U100 pad 37: unconnected-(U1-GPIO40/MTDO-Pad37) -> PCF8563_INT
- U100 pad 42: unconnected-(U1-GPIO44/U0RXD-Pad42) -> UART_RX
- U100 pad 43: unconnected-(U1-GPIO43/U0TXD-Pad43) -> UART_TX
- U101 pad 1: unconnected-(U3-TX-Pad1) -> RADAR_RX_PIN
- U101 pad 2: unconnected-(U3-RX-Pad2) -> RADAR_TX_PIN
- U101 pad 3: unconnected-(U3-OUT-Pad3) -> Net-(D105-A)
- U101 pad 4: unconnected-(U3-GND-Pad4) -> GND
- U101 pad 5: unconnected-(U3-VCC-Pad5) -> /esp32-s3/LD2410_VCC
- U102 pad 1: unconnected-(Brd1-GND-Pad1) -> GND
- U102 pad 2: unconnected-(Brd1-VCC-Pad2) -> +3.3V
- U102 pad 3: unconnected-(Brd1-SCL-Pad3) -> I2C_SCL
- U102 pad 4: unconnected-(Brd1-SDA-Pad4) -> I2C_SDA
- U103 pad 1: unconnected-(U2-SDA-Pad1) -> I2C_SCL
- U103 pad 2: unconnected-(U2-SCL-Pad2) -> I2C_SDA
- U103 pad 3: unconnected-(U2-GND-Pad3) -> GND
- U103 pad 4: unconnected-(U2-VIN-Pad4) -> +3.3V

Commit message: PCB initial layout
Parts:
- moved R302 251.7 mm to (279.2, 150.0), turned to 90 degrees
- moved U300 250.4 mm to (265.8, 155.0), turned to 180 degrees
- moved R300 246.8 mm to (267.8, 158.5)
- moved R301 242.6 mm to (264.0, 158.5)
- moved D302 240.3 mm to (276.0, 148.8), turned to 180 degrees
- moved C301 240.2 mm to (259.8, 155.0), turned to -90 degrees
- moved C303 239.3 mm to (269.2, 155.0), turned to -90 degrees
- moved C300 239.1 mm to (257.2, 155.0), turned to -90 degrees
- moved C304 237.6 mm to (267.8, 160.5), turned to 180 degrees
- moved L300 236.7 mm to (258.5, 152.2)
- moved C302 234.4 mm to (262.2, 155.0), turned to -90 degrees
- moved J300 234.4 mm to (238.8, 159.3), turned to 180 degrees
- moved J301 226.9 mm to (250.2, 149.3)
- moved D301 224.7 mm to (250.2, 155.1)
- moved D300 222.8 mm to (241.2, 162.8)
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Connections:
- net Net-(D401-A) renamed /PCF8563/VBAT
- net Net-(D401-K) renamed /PCF8563/PCF_VDD
- net Net-(U400-OSCI) renamed /PCF8563/OSCI
- U400 pad 2: GND -> /PCF8563/OSCO
- Y400 pad 3: GND -> /PCF8563/OSCO
Other:
- rule pad_to_mask_clearance: 0 -> 0.038

Commit message: Components can not fit 10x10 board
Parts:
- moved J100 203.9 mm to (191.2, 43.9), turned to 180 degrees
- moved R102 188.2 mm to (199.2, 71.9), turned to 90 degrees
- moved D103 185.2 mm to (199.2, 75.9), turned to -90 degrees
- moved R100 179.5 mm to (194.4, 71.9), turned to 90 degrees
- moved D101 176.4 mm to (194.4, 75.9), turned to -90 degrees
- moved C101 174.1 mm to (190.9, 70.9), turned to 180 degrees
- moved C100 172.1 mm to (190.9, 73.1), turned to 180 degrees
- moved D100 170.1 mm to (190.9, 75.6), turned to 180 degrees
- moved R101 166.0 mm to (186.9, 71.9), turned to 90 degrees
- moved D102 162.6 mm to (186.9, 75.9), turned to -90 degrees
- moved R103 161.1 mm to (184.2, 71.9), turned to 90 degrees
- moved D104 157.6 mm to (184.2, 75.9), turned to -90 degrees
- moved R107 149.9 mm to (254.2, 60.5)
- moved R108 149.9 mm to (254.2, 68.8)
- moved R109 149.9 mm to (254.2, 77.0)
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Other:
- board outline added: 100 x 100 mm

Commit message: minor PCB updates
Parts:
- added H1: MountingHole, MountingHole:MountingHole_3.2mm_M3, F.Cu at (30.0, 30.0)
- added H2: MountingHole, MountingHole:MountingHole_3.2mm_M3, F.Cu at (120.0, 30.0)
- added H3: MountingHole, MountingHole:MountingHole_3.2mm_M3, F.Cu at (120.0, 120.0)
- added H4: MountingHole, MountingHole:MountingHole_3.2mm_M3, F.Cu at (30.0, 120.0)
- BT400: moved to B.Cu
- moved J301 238.9 mm to (42.5, 29.2)
- moved D301 237.0 mm to (44.8, 35.0)
- moved D300 232.0 mm to (43.5, 39.4), turned to -90 degrees
- moved J300 231.3 mm to (40.0, 39.0), turned to -90 degrees
- moved R302 218.0 mm to (97.8, 27.2)
- moved D302 216.5 mm to (94.5, 28.8)
- moved C300 198.7 mm to (98.5, 33.5)
- moved C301 198.7 mm to (101.0, 33.5)
- moved L300 198.7 mm to (99.8, 30.7)
- moved C304 197.6 mm to (109.2, 40.5)
- moved R300 197.6 mm to (109.2, 38.5)
- moved R301 197.6 mm to (105.5, 38.5)
- moved C302 197.3 mm to (103.8, 35.5)
- moved C303 197.3 mm to (110.8, 35.5)
- moved L301 197.3 mm to (107.2, 29.4)
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Other:
- outline, holes or cut-outs redrawn

Commit message: Split scheme to 2 boards
Parts:
- removed D200, D201, D202, D203, D204, D205, D206, D207, D208, D209, D210, D211, D212, D213, D214, D215, D216, D217, D218, D219, D220, D221, D222, D223, D224, D225, D226, D227, D228, D229, D230, D231, D232, D233, D234, D235, D236, D237, D238, D239, D240, D241, D242, D243, D244, D245, D246, D247, D248, D249, D250, D251, D252, D253, D254, D255, D256, D257, D258, D259: WS2812B-2020, LED_SMD:LED_WS2812B-2020_PLCC4_2.0x2.0mm
- J101, J102, J103: footprint Connector_PinHeader_1.27mm:PinHeader_1x04_P1.27mm_Vertical -> Connector_PinHeader_2.54mm:PinHeader_1x04_P2.54mm_Vertical
- moved J100 206.8 mm to (30.6, 97.6), turned to -90 degrees
- moved R102 180.8 mm to (58.6, 89.6), turned to 180 degrees
- moved R100 176.6 mm to (58.6, 94.3), turned to 180 degrees
- moved D103 176.4 mm to (62.7, 89.6), turned to 0 degrees
- moved C101 174.7 mm to (57.6, 97.8), turned to -90 degrees
- moved C100 172.2 mm to (59.9, 97.8), turned to -90 degrees
- moved D101 172.1 mm to (62.6, 94.3), turned to 0 degrees
- moved R101 170.2 mm to (58.6, 101.8), turned to 180 degrees
- moved D100 169.3 mm to (62.4, 97.8), turned to -90 degrees
- moved R103 168.0 mm to (58.6, 104.6), turned to 180 degrees
- moved D102 165.7 mm to (62.6, 101.8), turned to 0 degrees
- moved D104 163.4 mm to (62.6, 104.6), turned to 0 degrees
- moved R107 161.9 mm to (40.0, 123.8), turned to 0 degrees
- moved SW101 155.6 mm to (36.5, 116.5)
- moved SW103 148.6 mm to (61.5, 116.5)
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